Commit message: backup

File: human_description/urdf/arm.xacro (robot description, xacro)
@@ -1,128 +1,135 @@
-<?xml version="1.0" ?>
-<robot name="left_arm" xmlns:xacro="http://playerstage.sourceforge.net/gazebo/xmlschema/#interface">
-  <material name="blue">
-    <color rgba="0 0 0.8 1"/>
-  </material>
-  <material name="black">
-    <color rgba="0 0 0 1"/>
-  </material>
-  <material name="white">
-    <color rgba="1 1 1 1"/>
-  </material>
-  <xacro:include filename="$(find my_robot_manipulator)/urdf/spherical.urdf.xacro"/>
+<?xml version="1.0" encoding="UTF-8"?>
+<!--URDF consist of two main parts: visual and inertial. In here I have only visual part -->
+<robot name="myhuman" xmlns:xacro="http://playerstage.sourceforge.net/gazebo/xmlschema/#interface">
+  <!-- Constants for human dimensions -->
+  <xacro:property name="PI" value="3.1415926535897931"/>
+  <xacro:property name="mass" value="1" /> <!-- arbitrary value for mass -->
+  <xacro:property name="width" value="0.1" /> <!-- Square dimensions (widthxwidth) of beams -->
+  <xacro:property name="length_upperarm" value=".35" /> <!-- Link 1 -->
+  <xacro:property name="length_forearm" value="1" /> <!-- Link 2 -->
+  <xacro:property name="length_hand" value="1" /> <!-- Link 3 -->
+  <xacro:property name="camera_link" value="0.05" /> <!-- Size of square 'camera' box Attach to head after-->
+  <!-- Import all Gazebo-customization elements, including Gazebo colors -->
+  <xacro:include filename="$(find ur5_with_hand_moveit_config)/human_description/urdf/human_arm.gazebo" />
+  <!-- Import Rviz colors -->
+  <xacro:include filename="$(find ur5_with_hand_moveit_config)/human_description/urdf/materials.xacro" />
+  <!-- Import Spherical joint macro -->
+  <xacro:include filename="$(find ur5_with_hand_moveit_config)/human_description/urdf/spherical.urdf.xacro"/>
+  <xacro:include filename="$(find ur5_with_hand_moveit_config)/human_description/urdf/spherical.urdf.xacro"/>
   <create/>
+  <link name="world"/>
+  <joint name="world_joint" type="fixed">
+    <parent link="world"/>
+    <child link="base_link"/>
+    <origin rpy="0.0 0.0 0.0" xyz="0.0 -1.0 1.0"/>
+  </joint>
   <link name="base_link">
     <visual>
       <origin rpy="0 0 0" xyz="0 0 0"/>
       <geometry>
-        <sphere radius="0.1"/>
+        <sphere radius="0.5"/>
       </geometry>
       <material name="white"/>
     </visual>
   </link>
-  <link name="human/shoulder_center">
-    <visual>
-      <origin rpy="0 0 0" xyz="0 0 0.050635057485"/>
-      <geometry>
-        <cylinder length="0.10127011497" radius="0.181172520845"/>
-      </geometry>
-    </visual>
-  </link>
-  <joint name="shoulder_center" type="fixed">
+  <xacro:spherical name="joint_1" parent="base_link" child="link_01">
     <origin rpy="0 0 0" xyz="0 0 0"/>
-    <parent link="base_link"/>
-    <child link="human/shoulder_center"/>
-  </joint>
-  <link name="human/left_arm_mount"/>
-  <link name="human/left_shoulder_0"/>
-  <link name="human/left_shoulder_1"/>
-  <link name="human/left_shoulder">
-    <visual>
-      <origin rpy="0 1.57079632679 0" xyz="0.147075804738 0 0"/>
-      <geometry>
-        <cylinder length="0.294151609476" radius="0.05"/>
-      </geometry>
-    </visual>
-  </link>
-  <link name="human/left_elbow">
-    <visual>
-      <origin rpy="0 1.57079632679 0" xyz="0.137074736994 0 0"/>
-      <geometry>
-        <cylinder length="0.274149473988" radius="0.025"/>
-      </geometry>
-    </visual>
-  </link>
-  <link name="human/left_wrist_0"/>
-  <link name="human/left_wrist_1"/>
-  <link name="human/left_wrist">
-    <visual>
-      <origin rpy="0 0 0" xyz="0.05 0 0"/>
-      <geometry>
-        <box size="0.1 0.05 .005"/>
-      </geometry>
-    </visual>
-  </link>
-  <link name="human/left_hand"/>
-  <!-- Joints -->
-  <joint name="left_arm_mount" type="fixed">
-    <origin rpy="0 0 1.57079632679" xyz="0 0.181172520845 -0.00609526854636"/>
-    <parent link="human/shoulder_center"/>
-    <child link="human/left_arm_mount"/>
-  </joint>
-  <!-- SHOULDER : spherical -->
-  <joint name="left_shoulder_0" type="revolute">
-    <origin rpy="0 0 0" xyz="0 0 0"/>
-    <axis xyz="0 1 0"/>
-    <parent link="human/left_arm_mount"/>
-    <child link="human/left_shoulder_0"/>
-    <limit effort="1" lower="-1.57079632679" upper="1.57079632679" velocity="1"/>
-  </joint>
-  <joint name="left_shoulder_1" type="revolute">
-    <origin rpy="0 0 0" xyz="0 0 0"/>
-    <axis xyz="0 0 1"/>
-    <parent link="human/left_shoulder_0"/>
-    <child link="human/left_shoulder_1"/>
-    <limit effort="1" lower="-2.35619449019" upper="1.57079632679" velocity="1"/>
-  </joint>
-  <joint name="left_shoulder_2" type="revolute">
-    <origin rpy="0 0 0" xyz="0 0 0"/>
-    <axis xyz="1 0 0"/>
-    <parent link="human/left_shoulder_1"/>
-    <child link="human/left_shoulder"/>
-    <limit effort="1" lower="-1.57079632679" upper="1.57079632679" velocity="1"/>
-  </joint>
-  <!-- END SHOULDER -->
-  <joint name="left_elbow_0" type="revolute">
-    <origin rpy="0 0 0" xyz="0.294151609476 0 0"/>
-    <axis xyz="0 0 1"/>
-    <parent link="human/left_shoulder"/>
-    <child link="human/left_elbow"/>
-    <limit effort="1" lower="-3.14159265359" upper="0.0" velocity="1"/>
-  </joint>
-  <joint name="left_wrist_0" type="revolute">
-    <origin rpy="0 0 0" xyz="0.274149473988 0 0"/>
-    <axis xyz="0 1 0"/>
-    <parent link="human/left_elbow"/>
-    <child link="human/left_wrist_0"/>
-    <limit effort="1" lower="-0.78539816339" upper="0.78539816339" velocity="1"/>
-  </joint>
-  <joint name="left_wrist_1" type="revolute">
-    <origin rpy="0 0 0" xyz="0 0 0"/>
-    <axis xyz="0 0 1"/>
-    <parent link="human/left_wrist_0"/>
-    <child link="human/left_wrist_1"/>
-    <limit effort="1" lower="-1.57079632679" upper="1.57079632679" velocity="1"/>
-  </joint>
-  <joint name="left_wrist_2" type="revolute">
-    <origin rpy="0 0 0" xyz="0 0 0"/>
-    <axis xyz="1 0 0"/>
-    <parent link="human/left_wrist_1"/>
-    <child link="human/left_wrist"/>
-    <limit effort="1" lower="-1.57079632679" upper="1.57079632679" velocity="1"/>
-  </joint>
-  <joint name="left_hand" type="fixed">
-    <origin rpy="0 0 0" xyz="0.1 0 0"/>
-    <parent link="human/left_wrist"/>
-    <child link="human/left_hand"/>
-  </joint>
+  </xacro:spherical>
+    <link name="link_01">
+      <visual>
+        <origin rpy="0 0 0" xyz="0 0 1.5"/>
+        <geometry>
+          <cylinder radius="0.5" length="3.0"/>
+        </geometry>
+        <material name="blue"/>
+      </visual>
+    </link>
+    <joint name="joint_2_ball" type="fixed">
+      <origin rpy="0 0 0" xyz="0 0 3.0"/>
+      <parent link="link_01"/>
+      <child link="link_02_ball"/>
+    </joint>
+    <link name="link_02_ball">
+      <visual>
+        <origin rpy="0 1.57 0" xyz="0 0 0"/>
+        <geometry>
+          <cylinder radius="0.25" length="0.5"/>
+        </geometry>
+        <material name="white"/>
+      </visual>
+    </link>
+    <joint name="joint_2" type="revolute">
+      <axis xyz="-1 0 0"/> <!-- rotate around z-axis-->
+      <limit effort="1000.0" lower="-3.14" upper="3.14" velocity="0.5"/>
+      <origin rpy="0 0 0" xyz="0 0 0"/>
+      <parent link="link_02_ball"/>
+      <child link="link_02"/>
+    </joint>
+    <link name="link_02">
+      <visual>
+        <origin rpy="0 0 0" xyz="0 0 1.0"/>
+        <geometry>
+          <cylinder radius="0.25" length="2.0"/>
+        </geometry>
+        <material name="blue"/>
+      </visual>
+    </link>
+    <joint name="joint_3_ball" type="fixed">
+      <origin rpy="0 0 0" xyz="0 0 2.0"/>  <!-- half of the height of the box 0.5-->
+      <parent link="link_02"/>
+      <child link="link_03_ball"/>
+    </joint>
+    <link name="link_03_ball">
+      <visual>
+        <origin rpy="0 0 0" xyz="0 0 0"/>
+        <geometry>
+          <sphere radius="0.12"/>
+        </geometry>
+        <material name="white"/>
+      </visual>
+    </link>
+    <xacro:spherical name="joint_3" parent="link_03_ball" child="link_03">
+      <origin rpy="0 0 0" xyz="0 0 0"/>
+    </xacro:spherical>
+    <link name="link_03">
+      <visual>
+        <origin rpy="0 0 0" xyz="0 0 0.5"/>
+        <geometry>
+          <cylinder radius="0.13" length="1"/>
+        </geometry>
+        <material name="blue"/>
+      </visual>
+    </link>
+    <joint name="link_03__gripper_a" type="prismatic">
+      <axis xyz="1 0 0"/> <!-- move around z-axis-->
+      <limit effort="1000.0" lower="0" upper="1.0" velocity="0.5"/>
+      <origin rpy="0 0 0" xyz="0 0 1.0"/>  <!-- half of the height of the box 0.5-->
+      <parent link="link_03"/>
+      <child link="gripper_a"/>
+    </joint>
+    <joint name="link_03__gripper_b" type="prismatic">
+      <axis xyz="-1 0 0"/> <!-- move around z-axis-->
+      <limit effort="1000.0" lower="0" upper="1.0" velocity="0.5"/>
+      <origin rpy="0 0 0" xyz="0 0 1.0"/>  <!-- half of the height of the box 0.5-->
+      <parent link="link_03"/>
+      <child link="gripper_b"/>
+    </joint>
+    <link name="gripper_a">
+      <visual>
+        <origin rpy="0 0 0" xyz="0.1 0 0.3"/>
+        <geometry>
+          <box size="0.2 0.2 0.6"/>
+        </geometry>
+        <material name="white"/>
+      </visual>
+    </link>
+    <link name="gripper_b">
+      <visual>
+        <origin rpy="0 0 0" xyz="-0.1 0 0.3"/>
+        <geometry>
+          <box size="0.2 0.2 0.6"/>
+        </geometry>
+        <material name="white"/>
+      </visual>
+    </link>
 </robot>

File: human_description/urdf/human_arm.xacro (robot description, xacro)
@@ -1,72 +1,108 @@
-<?xml version="1.0" encoding="UTF-8"?>
-<!--URDF consist of two main parts: visual and inertial. In here I have only visual part -->
-<robot name="mrm" xmlns:xacro="http://www.ros.org/wiki/xacro">
-  <link name="base_link">
+<?xml version="1.0" ?>
+<robot name="myhuman" xmlns:xacro="http://www.ros.org/wiki/xacro">
+  <!-- Constants for human dimensions -->
+  <xacro:property name="PI" value="3.1415926535897931"/>
+  <xacro:property name="mass" value="1" /> <!-- arbitrary value for mass -->
+  <xacro:property name="width" value="0.1" /> <!-- Square dimensions (widthxwidth) of beams -->
+  <xacro:property name="human_offset" value="0.0 0.0 0.0" /> <!-- Square dimensions (widthxwidth) of beams -->
+  <xacro:property name="length_upperarm" value=".35" /> <!-- Link 1 -->
+  <xacro:property name="length_forearm" value="0.3" /> <!-- Link 2 -->
+  <xacro:property name="length_hand" value="0.1" /> <!-- Link 3 -->
+  <xacro:property name="length_finger" value="0.05" /> <!-- Link 3 -->
+  <xacro:property name="camera_link" value="0.05" /> <!-- Size of square 'camera' box Attach to head after-->
+  <!-- Import all Gazebo-customization elements, including Gazebo colors -->
+  <xacro:include filename="$(find ur5_with_hand_moveit_config)/human_description/urdf/human_arm.gazebo" />
+  <!-- Import Rviz colors -->
+  <xacro:include filename="$(find ur5_with_hand_moveit_config)/human_description/urdf/materials.xacro" />
+  <!-- Import Spherical joint macro -->
+  <xacro:include filename="$(find ur5_with_hand_moveit_config)/human_description/urdf/spherical.urdf.xacro"/>
+  <xacro:include filename="$(find ur5_with_hand_moveit_config)/human_description/urdf/spherical.urdf.xacro"/>
+  <create/>
+  <link name="world"/>
+  <joint name="world_joint" type="fixed">
+    <parent link="world"/>
+    <child link="human_torso"/>
+    <origin rpy="0.0 0.0 0.0" xyz="${human_offset}"/>
+  </joint>
+  <link name="human_torso">
     <visual>
       <origin rpy="0 0 0" xyz="0 0 0"/>
       <geometry>
-        <box size="1 1 1"/>
+        <sphere radius="0.05"/>
       </geometry>
+      <material name="white"/>
     </visual>
   </link>
-  <joint name="base_link__link_01" type="revolute">
-    <axis xyz="1 0 0"/> <!-- rotate around z-axis-->
-    <limit effort="1000.0" lower="-3.14" upper="3.14" velocity="0.5"/>
-    <origin rpy="0 0 0" xyz="0 0 0.5"/>  <!-- half of the height of the box 0.5-->
-    <parent link="base_link"/>
-    <child link="link_01"/>
-  </joint>
-  <link name="link_01">
-    <visual>
-      <origin rpy="0 0 0" xyz="0 0 0.2"/>
-      <geometry>
-        <cylinder radius="0.35" length="0.4"/>
-      </geometry>
-    </visual>
-  </link>
-  <joint name="link_01__link_02" type="revolute">
-    <axis xyz="1 0 0"/> <!-- rotate around z-axis-->
-    <limit effort="1000.0" lower="-3.14" upper="3.14" velocity="0.5"/>
-    <origin rpy="0 0 0" xyz="0 0 0.4"/>  <!-- half of the height of the box 0.5-->
-    <parent link="link_01"/>
-    <child link="link_02"/>
-  </joint>
-  <link name="link_02">
-    <visual>
-      <origin rpy="0 0 0" xyz="0 0 0.2"/>
-      <geometry>
-        <cylinder radius="0.15" length="0.4"/>
-      </geometry>
-    </visual>
-  </link>
-  <joint name="link_02__gripper_a" type="prismatic">
-    <axis xyz="1 0 0"/> <!-- move around z-axis-->
-    <limit effort="1000.0" lower="0" upper="1.0" velocity="0.5"/>
-    <origin rpy="0 0 0" xyz="0 0 0.4"/>  <!-- half of the height of the box 0.5-->
-    <parent link="link_02"/>
-    <child link="gripper_a"/>
-  </joint>
-  <joint name="link_02__gripper_b" type="prismatic">
-    <axis xyz="-1 0 0"/> <!-- move around z-axis-->
-    <limit effort="1000.0" lower="0" upper="1.0" velocity="0.5"/>
-    <origin rpy="0 0 0" xyz="0 0 0.4"/>  <!-- half of the height of the box 0.5-->
-    <parent link="link_02"/>
-    <child link="gripper_b"/>
-  </joint>
-  <link name="gripper_a">
-    <visual>
-      <origin rpy="0 0 0" xyz="0.1 0 0.3"/>
-      <geometry>
-        <box size="0.2 0.2 0.6"/>
-      </geometry>
-    </visual>
-  </link>
-  <link name="gripper_b">
-    <visual>
-      <origin rpy="0 0 0" xyz="-0.1 0 0.3"/>
-      <geometry>
-        <box size="0.2 0.2 0.6"/>
-      </geometry>
-    </visual>
-  </link>
+  <xacro:spherical name="human_shoulder_joint" parent="human_torso" child="human_upperarm_link">
+    <origin rpy="0 0 0" xyz="0 0 0"/>
+  </xacro:spherical>
+    <link name="human_upperarm_link">
+      <visual>
+        <origin rpy="0 0 0" xyz="0 0 ${length_upperarm*0.5}"/>
+        <geometry>
+          <cylinder radius="${length_upperarm*0.1}" length="${length_upperarm}"/>
+        </geometry>
+        <material name="blue"/>
+      </visual>
+    </link>
+    <joint name="human_elbow_joint" type="revolute">
+      <axis xyz="-1 0 0"/> <!-- rotate around z-axis-->
+      <limit effort="1000.0" lower="-3.14" upper="3.14" velocity="0.5"/>
+      <origin rpy="0 0 0" xyz="0 0 ${length_upperarm}"/>
+      <parent link="human_upperarm_link"/>
+      <child link="human_forearm_link"/>
+    </joint>
+    <link name="human_forearm_link">
+      <visual>
+        <origin rpy="0 0 0" xyz="0 0 ${length_forearm*0.5}"/>
+        <geometry>
+          <cylinder radius="${length_forearm*0.1}" length="${length_forearm}"/>
+        </geometry>
+        <material name="blue"/>
+      </visual>
+    </link>
+    <xacro:spherical name="human_wrist_joint" parent="human_forearm_link" child="human_hand_link">
+      <origin rpy="0 0 0" xyz="0 0 0"/>
+    </xacro:spherical>
+    <link name="human_hand_link">
+      <visual>
+        <origin rpy="0 0 0" xyz="0 0 ${length_hand*0.5}"/>
+        <geometry>
+          <cylinder radius="${length_hand*0.1}" length="${length_hand}"/>
+        </geometry>
+        <material name="blue"/>
+      </visual>
+    </link>
+    <joint name="hand_to_finger1_joint" type="prismatic">
+      <axis xyz="1 0 0"/> <!-- move around z-axis-->
+      <limit effort="1000.0" lower="0" upper="1.0" velocity="0.5"/>
+      <origin rpy="0 0 0" xyz="0 0 ${length_hand}"/>  <!-- half of the height of the box 0.5-->
+      <parent link="human_hand_link"/>
+      <child link="human_finger1_link"/>
+    </joint>
+    <joint name="hand_to_finger2_joint" type="prismatic">
+      <axis xyz="-1 0 0"/> <!-- move around z-axis-->
+      <limit effort="1000.0" lower="0" upper="1.0" velocity="0.5"/>
+      <origin rpy="0 0 0" xyz="0 0 ${length_hand}"/>  <!-- half of the height of the box 0.5-->
+      <parent link="human_hand_link"/>
+      <child link="human_finger2_link"/>
+    </joint>
+    <link name="human_finger1_link">
+      <visual>
+        <origin rpy="0 0 0" xyz="${length_hand*0.1} 0 ${length_finger*0.5}"/>
+        <geometry>
+          <box size="${length_finger*0.3} ${length_finger*0.3} ${length_finger}"/>
+        </geometry>
+        <material name="white"/>
+      </visual>
+    </link>
+    <link name="human_finger2_link">
+      <visual>
+        <origin rpy="0 0 0" xyz="${-length_hand*0.1} 0 ${length_finger*0.5}"/>
+        <geometry>
+          <box size="${length_finger*0.3} ${length_finger*0.3} ${length_finger}"/>
+        </geometry>
+        <material name="white"/>
+      </visual>
+    </link>
 </robot>
